File: KiCad/Modulo LIFI/Modulo LIFI.kicad_sch (KiCad schematic)
At the start: 8 parts, among them J2 Arduino NANO, U3 LM358

Commit message: Mensaje describiendo tus cambios
Parts:
- removed R2, R3: 100k, Resistor_SMD:R_0805_2012Metric_Pad1.20x1.40mm_HandSolder, symbol Device:R_US
- C1: value 100nf -> 22pf
- R4: value 22k -> 1Mhoms
Connections:
- net GND: now also D2.2 (A), U3.3 (+)
Other:
- moved on the sheet: C2, D2, J2

Commit message: Mensaje describiendo tus cambios
Parts:
- C1: value 22pf -> 1nf
- R4: value 1Mhoms -> 680Khoms
Changed lines of the file:
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@@
 			)
 		)
-		(property "Value" "1Mhoms"
+		(property "Value" "680Khoms"
 			(at 213.36 62.23 90)
 			(effects
@@
 			)
 		)
-		(property "Value" "22pf"
+		(property "Value" "1nf"
 			(at 213.36 46.99 90)
 			(effects
