File: KiCad/Ant ESP8266/board.kicad_pcb (KiCad board)
At the start: 2 copper layers, 61.1 x 61.1 mm, 46 parts, among them P0 TCRT5000, P1 TCRT5000, P2 TCRT5000, P3 TCRT5000, P4 TCRT5000, P5 TCRT5000, P6 TCRT5000, P7 TCRT5000

Commit message: Actualizando documentos
Routing:
- net /<p>Proximity Sensors</p>/MUX_X3: track 2.77 -> 40.9 mm
- net AD0: track 5.48 -> 29.4 mm, vias 0 -> 1
- net /<p>MCU and Motors</p>/M_RIGHT_PWM: track 34.6 -> 56.4 mm, vias 0 -> 1
- net /<p>MCU and Motors</p>/E_LEFT_A: track 1.31 -> 16.2 mm
- net /<p>Proximity Sensors</p>/MUX_X5: track 18.1 -> 32.6 mm, vias 0 -> 2
- net Net-(LED0-DO): track 36.2 -> 50.6 mm, vias 0 -> 1
- net Net-(SWITCH0-O): track 6.54 -> 20.7 mm, vias 0 -> 3
- net /<p>MCU and Motors</p>/E_RIGHT_B: track 34.4 -> 48.0 mm, vias 0 -> 1
- net /<p>MCU and Motors</p>/E_RIGHT_A: track 5.89 -> 17.5 mm
- net Net-(R12-Pad2): track 6.26 -> 15.1 mm, vias 0 -> 1
- net Net-(CHRG0-PadC): track 3.20 -> 11.4 mm, vias 0 -> 1
- net Net-(SWITCH0-S): track 33.9 -> 40.7 mm, vias 0 -> 1
- net VCC: track 381.4 -> 386.7 mm, vias 1 -> 2
- net /<p>Proximity Sensors</p>/MUX_X2: track 0.00 -> 2.78 mm

Commit message: Descripción de los cambios
Parts:
- removed the C3 at (154.0, 97.9)
- removed MT3608: MT3608, board:MT3608
- turned MUX0 to 0 degrees
Routing:
- net /<p>Proximity Sensors</p>/MUX_X2: track 2.78 -> 60.1 mm
- net Net-(SWITCH0-S): track 40.7 -> 0.12 mm, vias 1 -> 0
- net /<p>Proximity Sensors</p>/MUX_X1: track 3.68 -> 42.3 mm
- net /<p>Proximity Sensors</p>/MUX_X6: track 3.16 -> 39.3 mm
- net /<p>Proximity Sensors</p>/MUX_X0: track 2.76 -> 34.1 mm
- net /<p>Proximity Sensors</p>/MUX_X4: track 4.09 -> 31.2 mm
- net /<p>Proximity Sensors</p>/MUX_X7: track 2.74 -> 29.1 mm
- net VCC: track 386.7 -> 401.8 mm, vias 2 -> 4
- net GND: track 0.00 -> 14.6 mm, vias 3 -> 8
- net MUX_A: track 0.00 -> 12.8 mm
- net MUX_B: track 0.00 -> 10.4 mm
- net /<p>Proximity Sensors</p>/MUX_X3: track 40.9 -> 31.6 mm
- net AD0: track 29.4 -> 21.3 mm
- net MUX_C: track 0.57 -> 7.29 mm, vias 1 -> 0
- net TP_B+: track 4.96 -> 0.00 mm
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
Commit message: Mensaje describiendo tus cambios
Parts:
- ESP-12E0: value ESP12E_DEVKIT -> ESP8266 ESP12E_DEVKIT
Other:
- board text added: "ANT"
- board text removed: "2023.10"
- board text removed: "HeRo"
- board text removed: "HeRo v2.7"
- board text removed: "ROS Compatible"
- board text removed: "verlab.dcc.ufmg.br"
Changed lines of the file:
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@@
 			)
 		)
-		(property "Value" "ESP12E_DEVKIT"
+		(property "Value" "ESP8266  ESP12E_DEVKIT"
 			(at 3.81 19.05 90)
 			(unlocked yes)
@@
 		)
 	)
-	(gr_text "HeRo"
-		(at 123.887005 92.549067 0)
-		(layer "F.SilkS")
-		(effects
-			(font
-				(size 0.93472 0.93472)
-				(thickness 0.08128)
-			)
-		)
-	)
 	(gr_text "A"
 		(at 168.974492 102.781995 90)
@@
 		)
 	)
-	(gr_text "verlab.dcc.ufmg.br"
-		(at 125.894496 93.722708 0)
-		(layer "F.SilkS")
-		(effects
-			(font
-				(size 0.560832 0.560832)
-				(thickness 0.048768)
-			)
-		)
-	)
 	(gr_text "A"
 		(at 128.674492 107.631995 90)
@@
 		)
 	)
-	(gr_text "2023.10"
-		(at 128.117214 92.703002 0)
-		(layer "F.SilkS")
-		(effects
-			(font
-				(size 0.70104 0.70104)
-				(thickness 0.06096)
-			)
-		)
-	)
 	(gr_text "+"
 		(at 169.254492 100.421995 0)
@@
 		)
 	)
-	(gr_text "HeRo\nv2.7"
-		(at 140.764492 131.231995 0)
-		(layer "F.SilkS")
-		(effects
-			(font
-				(size 1.40208 1.40208)
-				(thickness 0.12192)
-			)
-		)
-	)
 	(gr_text "GND"
 		(at 128.774492 103.131995 90)
@@
 		)
 	)
-	(gr_text "ROS\nCompatible"
-		(at 139.274492 78.731995 0)
-		(layer "F.SilkS")
-		(effects
-			(font
-				(size 1.1684 1.1684)
-				(thickness 0.1016)
-			)
-		)
-	)
-	(gr_text "verlab.dcc.ufmg.br"
-		(at 125.874496 93.702708 -0)
-		(layer "B.SilkS")
-		(effects
-			(font
-				(size 0.560832 0.560832)
-				(thickness 0.048768)
-			)
-			(justify mirror)
-		)
-	)
 	(gr_text "TCRT5000"
 		(at 151.517923 76.16543 -0)
@@
 		)
 	)
-	(gr_text "HeRo"
-		(at 148.124492 95.331995 -0)
+	(gr_text "ANT"
+		(at 148.124492 95.331995 0)
 		(layer "B.SilkS")
 		(effects
@@
 		)
 	)
-	(gr_text "2023.10"
-		(at 123.887214 92.683002 -0)
-		(layer "B.SilkS")
-		(effects
-			(font
-				(size 0.70104 0.70104)
-				(thickness 0.06096)
-			)
-			(justify mirror)
-		)
-	)
 	(gr_text "MUX             VCC"
 		(at 147.434492 106.361995 -0)
@@
 		)
 	)
-	(gr_text "HeRo"
-		(at 128.160142 92.574633 -0)
-		(layer "B.SilkS")
-		(effects
-			(font
-				(size 0.93472 0.93472)
-				(thickness 0.08128)
-			)
-			(justify mirror)
-		)
-	)
 	(gr_text "SCL     SDA   \nTX       RX     "
 		(at 142.914492 114.871995 0)
@@
 		)
 	)
-	(gr_text "ROS\nCompatible"
-		(at 139.324492 78.781995 -0)
-		(layer "B.SilkS")
-		(effects
-			(font
-				(size 1.1684 1.1684)
-				(thickness 0.1016)
-			)
-			(justify mirror)
-		)
-	)
-	(gr_text "HeRo\nv2.7"
-		(at 140.774492 131.231995 0)
-		(layer "B.SilkS")
-		(effects
-			(font
-				(size 1.40208 1.40208)
-				(thickness 0.12192)
-			)
-			(justify mirror)
-		)
-	)
