File: KiCad/Ant ESP8266/board_1.kicad_sch (KiCad schematic)
At the start: 6 parts

Commit message: Mensaje describiendo tus cambios
Parts:
- ESP-12E0: value ESP12E_DEVKIT -> ESP8266 ESP12E_DEVKIT
Other:
- moved on the sheet: E-HAT0
Changed lines of the file:
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@@
 	(wire
 		(pts
-			(xy 234.95 105.41) (xy 255.27 105.41)
-		)
-		(stroke
-			(width 0.1524)
-			(type solid)
-		)
-	)
-	(wire
-		(pts
-			(xy 234.95 102.87) (xy 247.65 102.87)
+			(xy 107.95 138.43) (xy 128.27 138.43)
+		)
+		(stroke
+			(width 0.1524)
+			(type solid)
+		)
+	)
+	(wire
+		(pts
+			(xy 107.95 135.89) (xy 120.65 135.89)
 		)
 		(stroke
@@
 	(wire
 		(pts
-			(xy 234.95 110.49) (xy 242.57 110.49)
+			(xy 107.95 143.51) (xy 115.57 143.51)
 		)
 		(stroke
@@
 	(wire
 		(pts
-			(xy 247.65 102.87) (xy 247.65 100.33)
-		)
-		(stroke
-			(width 0.1524)
-			(type solid)
-		)
-	)
-	(wire
-		(pts
-			(xy 180.34 101.6) (xy 200.66 101.6)
+			(xy 120.65 135.89) (xy 120.65 133.35)
+		)
+		(stroke
+			(width 0.1524)
+			(type solid)
+		)
+	)
+	(wire
+		(pts
+			(xy 180.34 101.6) (xy 195.58 101.6)
 		)
 		(stroke
@@
 	(wire
 		(pts
-			(xy 234.95 107.95) (xy 242.57 107.95)
+			(xy 107.95 140.97) (xy 115.57 140.97)
 		)
 		(stroke
@@
 	)
 	(label "SCL_TX"
-		(at 242.57 107.95 0)
+		(at 115.57 140.97 0)
 		(effects
 			(font
@@
 	)
 	(label "SDA_RX"
-		(at 242.57 110.49 0)
+		(at 115.57 143.51 0)
 		(effects
 			(font
@@
 	(symbol
 		(lib_id "board-eagle-import:supply1_371_GND")
-		(at 200.66 104.14 0)
+		(at 195.58 104.14 0)
 		(unit 1)
 		(exclude_from_sim no)
@@
 		(dnp no)
 		(property "Reference" "#GND5"
-			(at 200.66 104.14 0)
+			(at 195.58 104.14 0)
 			(effects
 				(font
@@
 		)
 		(property "Value" "GND"
-			(at 200.66 106.68 0)
+			(at 195.58 106.68 0)
 			(effects
 				(font
@@
 		)
 		(property "Footprint" ""
-			(at 200.66 104.14 0)
+			(at 195.58 104.14 0)
 			(effects
 				(font
@@
 		)
 		(property "Datasheet" ""
-			(at 200.66 104.14 0)
+			(at 195.58 104.14 0)
 			(effects
 				(font
@@
 		)
 		(property "Description" ""
-			(at 200.66 104.14 0)
+			(at 195.58 104.14 0)
 			(effects
 				(font
@@
 	(symbol
 		(lib_id "board-eagle-import:frames_229_A4L-LOC")
-		(at 21.59 196.85 0)
+		(at 271.78 137.16 0)
 		(unit 1)
 		(exclude_from_sim no)
@@
 		(dnp no)
 		(property "Reference" "#FRAME2"
-			(at 21.59 196.85 0)
+			(at 271.78 137.16 0)
 			(effects
 				(font
@@
 		)
 		(property "Value" "MCU and Motors Connectors"
-			(at 21.59 196.85 0)
+			(at 271.78 137.16 0)
 			(effects
 				(font
@@
 		)
 		(property "Footprint" ""
-			(at 21.59 196.85 0)
+			(at 271.78 137.16 0)
 			(effects
 				(font
@@
 		)
 		(property "Datasheet" ""
-			(at 21.59 196.85 0)
+			(at 271.78 137.16 0)
 			(effects
 				(font
@@
 		)
 		(property "Description" ""
-			(at 21.59 196.85 0)
+			(at 271.78 137.16 0)
 			(effects
 				(font
@@
 		)
 		(property "TITLE" "MCU and Motors"
-			(at 238.76 176.276 0)
+			(at 488.95 116.586 0)
 			(effects
 				(font
@@
 			)
 		)
-		(property "Value" "ESP12E_DEVKIT"
-			(at 153.67 82.55 0)
+		(property "Value" "ESP8266  ESP12E_DEVKIT"
+			(at 147.828 82.042 0)
 			(effects
 				(font
@@
 	(symbol
 		(lib_id "board-eagle-import:pinhead_PINHD-1X4")
-		(at 232.41 105.41 180)
+		(at 105.41 138.43 180)
 		(unit 1)
 		(exclude_from_sim no)
@@
 		(dnp no)
 		(property "Reference" "E-HAT0"
-			(at 237.1598 113.8428 0)
+			(at 110.1598 146.8628 0)
 			(effects
 				(font
@@
 		)
 		(property "Value" "PINHD-1X4"
-			(at 238.76 97.79 0)
+			(at 111.76 130.81 0)
 			(effects
 				(font
@@
 		)
 		(property "Footprint" "board:1X04"
-			(at 232.41 105.41 0)
+			(at 105.41 138.43 0)
 			(effects
 				(font
@@
 		)
 		(property "Datasheet" ""
-			(at 232.41 105.41 0)
+			(at 105.41 138.43 0)
 			(effects
 				(font
@@
 		)
 		(property "Description" ""
-			(at 232.41 105.41 0)
+			(at 105.41 138.43 0)
 			(effects
 				(font
@@
 	(symbol
 		(lib_id "board-eagle-import:supply1_371_VCC")
-		(at 247.65 97.79 0)
+		(at 120.65 130.81 0)
 		(unit 1)
 		(exclude_from_sim no)
@@
 		(dnp no)
 		(property "Reference" "#P+22"
-			(at 247.65 97.79 0)
+			(at 120.65 130.81 0)
 			(effects
 				(font
@@
 		)
 		(property "Value" "VCC"
-			(at 247.65 95.25 90)
+			(at 120.65 128.27 90)
 			(effects
 				(font
@@
 		)
 		(property "Footprint" ""
-			(at 247.65 97.79 0)
+			(at 120.65 130.81 0)
 			(effects
 				(font
@@
 		)
 		(property "Datasheet" ""
-			(at 247.65 97.79 0)
+			(at 120.65 130.81 0)
 			(effects
 				(font
@@
 		)
 		(property "Description" ""
-			(at 247.65 97.79 0)
+			(at 120.65 130.81 0)
 			(effects
 				(font
@@
 	(symbol
 		(lib_id "board-eagle-import:supply1_371_GND")
-		(at 255.27 107.95 0)
+		(at 128.27 140.97 0)
 		(unit 1)
 		(exclude_from_sim no)
@@
 		(dnp no)
 		(property "Reference" "#GND18"
-			(at 255.27 107.95 0)
+			(at 128.27 140.97 0)
 			(effects
 				(font
@@
 		)
 		(property "Value" "GND"
-			(at 257.81 110.49 0)
+			(at 130.81 143.51 0)
 			(effects
 				(font
@@
 		)
 		(property "Footprint" ""
-			(at 255.27 107.95 0)
+			(at 128.27 140.97 0)
 			(effects
 				(font
@@
 		)
 		(property "Datasheet" ""
-			(at 255.27 107.95 0)
+			(at 128.27 140.97 0)
 			(effects
 				(font
@@
 		)
 		(property "Description" ""
-			(at 255.27 107.95 0)
-			(effects
-				(font
+			(at 128.27 140.97 0)
+			(effects
+				(font
