File: KiCad/Ant ESP8266/board_2.kicad_sch (KiCad schematic)
At the start: 22 parts, among them P0 TCRT5000, P1 TCRT5000, P2 TCRT5000, P3 TCRT5000, P4 TCRT5000, P5 TCRT5000, P6 TCRT5000, P7 TCRT5000

Commit message: Mensaje describiendo tus cambios
Changed lines of the file:
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@@
 		)
 		(property "Value" "MOSFET-NREFLOW"
-			(at 155.41 144.97 0)
+			(at 155.194 146.05 0)
 			(effects
 				(font
