File: KiCad/Ant Raspberry PI PICO/board.kicad_pcb (KiCad board)
At the start: 2 copper layers, 61.1 x 61.1 mm, 51 parts, among them J1 Conn_01x20_MountingPin, J2 Conn_01x20_MountingPin, J3 Con, J4 Con, J5 Con, J6 Con, P0 TCRT5000, P1 TCRT5000, P2 TCRT5000, P3 TCRT5000, P4 TCRT5000, P5 TCRT5000, P6 TCRT5000, P7 TCRT5000, U1 Pico

Commit message: Descripción de los cambios
Routing:
- net VCC: track 412.0 -> 412.9 mm
- net /<p>MCU and Motors</p>/M_LEFT_PWM: track 22.6 -> 23.3 mm
- net Net-(SWITCH0-P): track 26.1 -> 26.7 mm
- net /<p>MCU and Motors</p>/M_RIGHT_PWM: track 59.2 -> 58.6 mm
Changed lines of the file:
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@@
 			(drillshape 0)
 			(scaleselection 1)
-			(outputdirectory "../Ant ESP8266/Gerber/")
+			(outputdirectory "Gcode/")
 		)
 	)
@@
 	)
 	(segment
-		(start 143.4838 105.6662)
-		(end 143.4838 114.925182)
-		(width 0.42)
-		(layer "F.Cu")
-		(net 2)
-	)
-	(segment
 		(start 166.925001 82.331995)
 		(end 166.925001 82.551995)
@@
 	)
 	(segment
-		(start 143.4838 114.925182)
-		(end 146.291809 117.733191)
+		(start 147.5 92.275)
+		(end 148.715 92.275)
 		(width 0.42)
 		(layer "F.Cu")
@@
 	)
 	(segment
-		(start 144.15 105)
-		(end 143.4838 105.6662)
-		(width 0.42)
-		(layer "F.Cu")
-		(net 2)
-	)
-	(segment
 		(start 170.456129 85.95363)
 		(end 170.456129 85.850361)
@@
 	)
 	(segment
+		(start 142.9 106.25)
+		(end 142.9 114.71)
+		(width 0.42)
+		(layer "F.Cu")
+		(net 2)
+	)
+	(segment
 		(start 119.52523 107.411258)
 		(end 119.524492 107.411995)
@@
 	)
 	(segment
+		(start 145.923191 117.733191)
+		(end 146.291809 117.733191)
+		(width 0.42)
+		(layer "F.Cu")
+		(net 2)
+	)
+	(segment
 		(start 172.355744 122.190744)
 		(end 169.545 119.38)
@@
 	)
 	(segment
+		(start 142.9 114.71)
+		(end 145.923191 117.733191)
+		(width 0.42)
+		(layer "F.Cu")
+		(net 2)
+	)
+	(segment
 		(start 143.6 96.795)
 		(end 143.6 97.375)
@@
 	)
 	(segment
+		(start 148.715 92.275)
+		(end 149.1 92.66)
+		(width 0.42)
+		(layer "F.Cu")
+		(net 2)
+	)
+	(segment
 		(start 122.486248 120.083752)
 		(end 119.524492 117.121995)
@@
 	)
 	(segment
+		(start 144.15 105)
+		(end 142.9 106.25)
+		(width 0.42)
+		(layer "F.Cu")
+		(net 2)
+	)
+	(segment
 		(start 142.24 78.105)
 		(end 142.24 76.021995)
@@
 	)
 	(segment
+		(start 149.1 92.66)
+		(end 149.1 92.985)
+		(width 0.42)
+		(layer "F.Cu")
+		(net 2)
+	)
+	(segment
 		(start 168.806995 114.831995)
 		(end 166.724492 114.831995)
@@
 	)
 	(segment
-		(start 147.5 92.275)
-		(end 148.39 92.275)
-		(width 0.42)
-		(layer "F.Cu")
-		(net 2)
-	)
-	(segment
 		(start 147.45 99.275)
 		(end 147.45 101.3)
@@
 	)
 	(segment
-		(start 148.39 92.275)
-		(end 149.1 92.985)
-		(width 0.42)
-		(layer "F.Cu")
-		(net 2)
-	)
-	(segment
 		(start 168.551532 121.755408)
 		(end 170.659492 123.863367)
@@
 	)
 	(segment
+		(start 170.16 108.25)
+		(end 171.19 109.28)
+		(width 0.42)
+		(layer "F.Cu")
+		(net 8)
+	)
+	(segment
 		(start 169.15 97.86)
 		(end 169.15 95.875)
@@
 	)
 	(segment
-		(start 171.19 110.265)
+		(start 169.175 108.25)
+		(end 170.16 108.25)
+		(width 0.42)
+		(layer "F.Cu")
+		(net 8)
+	)
+	(segment
+		(start 171.19 109.28)
 		(end 171.19 116.8)
 		(width 0.42)
@@
 		(net 8)
 	)
-	(segment
-		(start 169.175 108.25)
-		(end 171.19 110.265)
-		(width 0.42)
-		(layer "F.Cu")
-		(net 8)
-	)
 	(via
 		(at 169.175 108.25)
@@
 	)
 	(segment
-		(start 152.644968 84.925)
-		(end 153.304168 84.2658)
-		(width 0.42)
-		(layer "F.Cu")
-		(net 14)
-	)
-	(segment
-		(start 153.304168 84.2658)
+		(start 144.808048 84.2658)
 		(end 157.0208 84.2658)
 		(width 0.42)
@@
 	)
 	(segment
-		(start 136.1766 80.37)
-		(end 140.912248 80.37)
+		(start 140.912248 80.37)
+		(end 144.808048 84.2658)
 		(width 0.42)
 		(layer "F.Cu")
@@
 	)
 	(segment
-		(start 145.467248 84.925)
-		(end 152.644968 84.925)
-		(width 0.42)
-		(layer "F.Cu")
-		(net 14)
-	)
-	(segment
-		(start 140.912248 80.37)
-		(end 145.467248 84.925)
+		(start 136.1766 80.37)
+		(end 140.912248 80.37)
 		(width 0.42)
 		(layer "F.Cu")
@@
 	)
 	(segment
-		(start 166.724492 112.291995)
+		(start 163.311995 107.621995)
 		(end 162.054492 107.621995)
 		(width 0.508)
@@
 		(net 15)
 	)
+	(segment
+		(start 166.724492 112.291995)
+		(end 166.724492 111.034492)
+		(width 0.508)
+		(layer "F.Cu")
+		(net 15)
+	)
+	(segment
+		(start 166.724492 111.034492)
+		(end 163.311995 107.621995)
+		(width 0.508)
+		(layer "F.Cu")
+		(net 15)
+	)
 	(via
 		(at 162.054492 107.621995)
@@
 	)
 	(segment
-		(start 148.95 121.4)
-		(end 141.65 114.1)
+		(start 148.24 121.4)
+		(end 141.65 114.81)
 		(width 0.42)
 		(layer "F.Cu")
@@
 	)
 	(segment
-		(start 141.65 114.1)
+		(start 141.65 114.81)
 		(end 141.65 92.125)
 		(width 0.42)
@@
 		(net 20)
 	)
+	(segment
+		(start 148.95 121.4)
+		(end 148.24 121.4)
+		(width 0.42)
+		(layer "F.Cu")
+		(net 20)
+	)
 	(via
 		(at 148.95 121.4)
@@
 		(width 0.42)
 		(layer "F.Cu")
-		(net 22)
-	)
-	(segment
-		(start 160.925 85.675)
-		(end 161.0358 85.7858)
-		(width 0.42)
-		(layer "F.Cu")
