File: KiCad/Ant Raspberry PI PICO/board_1.kicad_sch (KiCad schematic)
At the start: 12 parts, among them J1 Conn_01x20_MountingPin, J2 Conn_01x20_MountingPin, J3 Con, J4 Con, J5 Con, J6 Con, U1 Pico

Commit message: Mensaje describiendo tus cambios
Other:
- moved on the sheet: E_LEFT0, E_RIGHT0
Changed lines of the file:
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@@
 	(wire
 		(pts
-			(xy 85.09 116.84) (xy 90.17 116.84)
+			(xy 85.09 113.03) (xy 90.17 113.03)
 		)
 		(stroke
@@
 	(wire
 		(pts
-			(xy 62.23 119.38) (xy 62.23 121.92)
+			(xy 62.23 115.57) (xy 62.23 118.11)
 		)
 		(stroke
@@
 	(wire
 		(pts
-			(xy 54.61 111.76) (xy 62.23 111.76)
+			(xy 54.61 107.95) (xy 62.23 107.95)
 		)
 		(stroke
@@
 	(wire
 		(pts
-			(xy 54.61 114.3) (xy 62.23 114.3)
+			(xy 54.61 110.49) (xy 62.23 110.49)
 		)
 		(stroke
@@
 	(wire
 		(pts
-			(xy 54.61 116.84) (xy 59.69 116.84)
+			(xy 54.61 113.03) (xy 59.69 113.03)
 		)
 		(stroke
@@
 	(wire
 		(pts
-			(xy 92.71 119.38) (xy 92.71 121.92)
+			(xy 92.71 115.57) (xy 92.71 118.11)
 		)
 		(stroke
@@
 	(wire
 		(pts
-			(xy 59.69 116.84) (xy 62.23 119.38)
+			(xy 59.69 113.03) (xy 62.23 115.57)
 		)
 		(stroke
@@
 	(wire
 		(pts
-			(xy 85.09 114.3) (xy 92.71 114.3)
+			(xy 85.09 110.49) (xy 92.71 110.49)
 		)
 		(stroke
@@
 	(wire
 		(pts
-			(xy 85.09 111.76) (xy 92.71 111.76)
+			(xy 85.09 107.95) (xy 92.71 107.95)
 		)
 		(stroke
@@
 	(wire
 		(pts
-			(xy 90.17 116.84) (xy 92.71 119.38)
+			(xy 90.17 113.03) (xy 92.71 115.57)
 		)
 		(stroke
@@
 	)
 	(label "E_RIGHT_A"
-		(at 62.23 111.76 0)
+		(at 62.23 107.95 0)
 		(effects
 			(font
@@
 	)
 	(label "E_LEFT_B"
-		(at 92.71 114.3 0)
+		(at 92.71 110.49 0)
 		(effects
 			(font
@@
 	)
 	(label "E_LEFT_A"
-		(at 92.71 111.76 0)
+		(at 92.71 107.95 0)
 		(effects
 			(font
@@
 	)
 	(label "E_RIGHT_B"
-		(at 62.23 114.3 0)
+		(at 62.23 110.49 0)
 		(effects
 			(font
@@
 	(symbol
 		(lib_id "board-eagle-import:pinhead_PINHD-1X3")
-		(at 52.07 114.3 180)
+		(at 52.07 110.49 180)
 		(unit 1)
 		(exclude_from_sim no)
@@
 		(dnp no)
 		(property "Reference" "E_RIGHT0"
-			(at 58.42 120.015 0)
+			(at 58.42 116.205 0)
 			(effects
 				(font
@@
 		)
 		(property "Value" "PINHD-1X3"
-			(at 58.42 106.68 0)
+			(at 58.42 102.87 0)
 			(effects
 				(font
@@
 		)
 		(property "Footprint" "board:1X03"
-			(at 52.07 114.3 0)
+			(at 52.07 110.49 0)
 			(effects
 				(font
@@
 		)
 		(property "Datasheet" ""
-			(at 52.07 114.3 0)
+			(at 52.07 110.49 0)
 			(effects
 				(font
@@
 		)
 		(property "Description" ""
-			(at 52.07 114.3 0)
+			(at 52.07 110.49 0)
 			(effects
 				(font
@@
 	(symbol
 		(lib_id "board-eagle-import:supply1_371_GND")
-		(at 92.71 124.46 0)
+		(at 92.71 120.65 0)
 		(unit 1)
 		(exclude_from_sim no)
@@
 		(dnp no)
 		(property "Reference" "#GND9"
-			(at 92.71 124.46 0)
+			(at 92.71 120.65 0)
 			(effects
 				(font
@@
 		)
 		(property "Value" "GND"
-			(at 95.25 127 0)
+			(at 95.25 123.19 0)
 			(effects
 				(font
@@
 		)
 		(property "Footprint" ""
-			(at 92.71 124.46 0)
+			(at 92.71 120.65 0)
 			(effects
 				(font
@@
 		)
 		(property "Datasheet" ""
-			(at 92.71 124.46 0)
+			(at 92.71 120.65 0)
 			(effects
 				(font
@@
 		)
 		(property "Description" ""
-			(at 92.71 124.46 0)
+			(at 92.71 120.65 0)
 			(effects
 				(font
@@
 	(symbol
 		(lib_id "board-eagle-import:pinhead_PINHD-1X3")
-		(at 82.55 114.3 180)
+		(at 82.55 110.49 180)
 		(unit 1)
 		(exclude_from_sim no)
@@
 		(dnp no)
 		(property "Reference" "E_LEFT0"
-			(at 88.9 120.015 0)
+			(at 88.9 116.205 0)
 			(effects
 				(font
@@
 		)
 		(property "Value" "PINHD-1X3"
-			(at 88.9 106.68 0)
+			(at 88.9 102.87 0)
 			(effects
 				(font
@@
 		)
 		(property "Footprint" "board:1X03"
-			(at 82.55 114.3 0)
+			(at 82.55 110.49 0)
 			(effects
 				(font
@@
 		)
 		(property "Datasheet" ""
-			(at 82.55 114.3 0)
+			(at 82.55 110.49 0)
 			(effects
 				(font
@@
 		)
 		(property "Description" ""
-			(at 82.55 114.3 0)
+			(at 82.55 110.49 0)
 			(effects
 				(font
@@
 	(symbol
 		(lib_id "board-eagle-import:supply1_371_GND")
-		(at 62.23 124.46 0)
+		(at 62.23 120.65 0)
 		(unit 1)
 		(exclude_from_sim no)
@@
 		(dnp no)
 		(property "Reference" "#GND8"
-			(at 62.23 124.46 0)
+			(at 62.23 120.65 0)
 			(effects
 				(font
@@
 		)
 		(property "Value" "GND"
-			(at 64.77 127 0)
+			(at 64.77 123.19 0)
 			(effects
 				(font
@@
 		)
 		(property "Footprint" ""
-			(at 62.23 124.46 0)
+			(at 62.23 120.65 0)
 			(effects
 				(font
@@
 		)
 		(property "Datasheet" ""
-			(at 62.23 124.46 0)
+			(at 62.23 120.65 0)
 			(effects
 				(font
@@
 		)
 		(property "Description" ""
-			(at 62.23 124.46 0)
-			(effects
-				(font
+			(at 62.23 120.65 0)
+			(effects
+				(font
