File: KiCad/Ant Raspberry PI PICO/board_2.kicad_sch (KiCad schematic)
At the start: 22 parts, among them P0 TCRT5000, P1 TCRT5000, P2 TCRT5000, P3 TCRT5000, P4 TCRT5000, P5 TCRT5000, P6 TCRT5000, P7 TCRT5000

Commit message: Mensaje describiendo tus cambios
Other:
- moved on the sheet: IRLML2502, P0, P1, P3, P5, R10, R11, R2, R3, R4, R5, R8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
